File: pcb-01.kicad_pcb (KiCad board)
At the start: 2 copper layers, 303.8 x 101.3 mm, 163 parts, among them J1 TYPE-C-31-M12_13, Q1 DTC123J, SW1 Esc, SW10 9, SW11 0, SW12 -, SW13 =, SW14 \, SW15 `, SW16 Home, SW17 Tab_150, SW18 Q, SW19 W, SW2 1, SW20 E, SW21 R, SW22 T, SW23 Y, SW24 U, SW25 I, SW26 O, SW27 P, SW28 [, SW29 ], SW3 2, SW30 Bkspc_150, SW31 Pgup, SW32 Caps_175, SW33 A, SW34 S, SW35 D, SW36 F, SW37 G, SW38 H, SW39 J, SW4 3, SW40 K, SW41 L, SW42 ;, SW43 ', SW44 Enter_225, SW45 Pgdwn, SW46 LShift_225, SW47 Z, SW48 X, SW49 C, SW5 4, SW50 V, SW51 B, SW52 N, SW53 M, SW54 <, SW55 >, SW56 ?, SW57 RShift_175, SW58 Up, SW59 Fn, SW6 5, SW60 LCtrl_150, SW61 LAlt_150, SW62 Space_7, SW63 RAlt_150, SW64 Left, SW65 Down, SW66 Right, SW67 SW_Push, SW68 Bkspc_200, SW69 Caps_125, SW7 6, SW8 7, SW9 8, U1 USBLC6-2SC6, U2 MCP1700-3002E_SOT23, U3 STM32F072CBTx

Commit message: updated pcb graphics
Parts:
- removed the G*** at (192.4, 138.4)
- removed the G*** at (132.4, 138.9)
- added G***: LOGO, logos:tagw, B.Cu at (193.8, 139.0)
- added G***: LOGO, logos:tagw, F.Cu at (131.7, 139.0)
- added G***: LOGO, logos:panda-logo, B.Cu at (131.6, 139.0)
- added G***: LOGO, logos:panda-logo, F.Cu at (194.0, 139.0)
Routing:
- net GND: track 58.1 -> 56.1 mm
- net Col11: track 317.5 -> 318.5 mm
Other:
- outline, holes or cut-outs redrawn
- board text removed: "things are going well by generic_panda"
