File: kicadfiles/pcb-01.kicad_pcb (KiCad board)
At the start: 2 copper layers, 303.8 x 101.3 mm, 165 parts, among them J1 TYPE-C-31-M12_13, Q1 DTC123J, SW1 Esc, SW10 9, SW11 0, SW12 -, SW13 =, SW14 \, SW15 `, SW16 Home, SW17 Tab_150, SW18 Q, SW19 W, SW2 1, SW20 E, SW21 R, SW22 T, SW23 Y, SW24 U, SW25 I, SW26 O, SW27 P, SW28 [, SW29 ], SW3 2, SW30 Bkspc_150, SW31 Pgup, SW32 Caps_175, SW33 A, SW34 S, SW35 D, SW36 F, SW37 G, SW38 H, SW39 J, SW4 3, SW40 K, SW41 L, SW42 ;, SW43 ', SW44 Enter_225, SW45 Pgdwn, SW46 LShift_225, SW47 Z, SW48 X, SW49 C, SW5 4, SW50 V, SW51 B, SW52 N, SW53 M, SW54 <, SW55 >, SW56 ?, SW57 RShift_175, SW58 Up, SW59 Fn, SW6 5, SW60 LCtrl_150, SW61 LAlt_150, SW62 Space_7, SW63 RAlt_150, SW64 Left, SW65 Down, SW66 Right, SW67 SW_Push, SW68 Bkspc_200, SW69 Caps_125, SW7 6, SW8 7, SW9 8, U1 USBLC6-2SC6, U2 MCP1700-3002E_SOT23, U3 STM32F072CBTx

Commit message: added polyfuse and updated routing
Parts:
- added F1: 500mA, Fuse:Fuse_1206_3216Metric, B.Cu at (54.0, 80.7)
- moved D67 0.15 mm to (51.6, 85.3)
Connections:
- C1 pad 1: VBUS -> Net-(C1-Pad1)
- D67 pad 1: VBUS -> Net-(C1-Pad1)
- R3 pad 1: VBUS -> Net-(C1-Pad1)
- U2 pad 3: VBUS -> Net-(C1-Pad1)
Routing:
- net VBUS: track 481.2 -> 465.6 mm
- net Net-(C1-Pad1): track 0.00 -> 13.3 mm
- net Row1: track 335.3 -> 342.5 mm
- net Row2: track 310.7 -> 315.4 mm
- net D+BUS: track 12.5 -> 10.2 mm
- net Col2: track 59.7 -> 58.1 mm
- net D+: track 174.1 -> 172.9 mm
- net D-BUS: track 10.1 -> 10.8 mm
- net Net-(J1-PadB5): track 3.87 -> 3.32 mm
- net Net-(J1-PadA5): track 3.86 -> 3.31 mm
