File: kicadfiles/pcb-01.sch (KiCad schematic (older format))
At the start: 161 parts, among them J1 TYPE-C-31-M12_13, Q1 DTC123J, SW1 Esc, SW10 9, SW11 0, SW12 -, SW13 =, SW14 \\, SW15 `, SW16 Home, SW17 Tab_150, SW18 Q, SW19 W, SW2 1, SW20 E, SW21 R, SW22 T, SW23 Y, SW24 U, SW25 I, SW26 O, SW27 P, SW28 [, SW29 ], SW3 2, SW30 Bkspc_150, SW31 Pgup, SW32 Caps_175, SW33 A, SW34 S, SW35 D, SW36 F, SW37 G, SW38 H, SW39 J, SW4 3, SW40 K, SW41 L, SW42 ;, SW43 ', SW44 Enter_225, SW45 Pgdwn, SW46 LShift_225, SW47 Z, SW48 X, SW49 C, SW5 4, SW50 V, SW51 B, SW52 N, SW53 M, SW54 <, SW55 >, SW56 ?, SW57 RShift_175, SW58 Up, SW59 Fn, SW6 5, SW60 LCtrl_150, SW61 LAlt_150, SW62 Space_7, SW63 RAlt_150, SW64 Left, SW65 Down, SW66 Right, SW67 SW_Push, SW68 Bkspc_200, SW69 Caps_125, SW7 6, SW8 7, SW9 8, U1 USBLC6-2SC6, U2 MCP1700-3002E_SOT23, U3 STM32F072CBTx

Commit message: added polyfuse and updated routing
Parts:
- added F1: 500mA, Fuse:Fuse_1206_3216Metric, symbol Device:Polyfuse_Small
- J1: symbol acheronSymbols:TYPE-C-31-M12_13 -> pcb-01-rescue:TYPE-C-31-M12_13-acheronSymbols
- Q1: symbol acheronSymbols:DTC123J -> pcb-01-rescue:DTC123J-acheronSymbols
- SW1, SW10, SW11, SW12, SW13, SW14, SW15, SW16, SW17, SW18, SW19, SW2, SW20, SW21, SW22, SW23, SW24, SW25, SW26, SW27, SW28, SW29, SW3, SW30, SW31, SW32, SW33, SW34, SW35, SW36, SW37, SW38, SW39, SW4, SW40, SW41, SW42, SW43, SW44, SW45, SW46, SW47, SW48, SW49, SW5, SW50, SW51, SW52, SW53, SW54, SW55, SW56, SW57, SW58, SW59, SW6, SW60, SW61, SW62, SW63, SW64, SW65, SW66, SW68, SW69, SW7, SW8, SW9: symbol acheronSymbols:MXSwitch -> pcb-01-rescue:MXSwitch-acheronSymbols
Connections:
- net VBUS: now also F1.2; no longer C1.1, D67.1 (K), R3.1, U2.3 (VI)
- new net: C1.1, D67.1 (K), F1.1, R3.1, U2.3 (VI)
